File: kicad/cycloscope/ cycloscope_photo_trigger.sch (KiCad schematic (older format))
At the start: 19 parts, among them IC1 ATMEGA328P-P, P1 CONN_1, P2 CONN_1, P3 CONN_1, P4 CONN_1, P5 CONN_2, P6 CONN_6, P7 CONN_5, P8 CONN_2, SW1 SW_PUSH

Commit message: Aggiornato software e schemi kicad
Parts:
- removed P7: CONN_5, symbol CONN_5
- added J1: JACK_3.5MM_3PIN, symbol JACK_3.5MM_3PIN
Connections:
- wire segments 49 -> 46
- no-connect marks 18 -> 19
Changed lines of the file:
@@
-EESchema Schematic File Version 2  date Mon 21 Apr 2014 19:16:43 CEST
+EESchema Schematic File Version 2  date Fri 25 Apr 2014 22:11:27 CEST
 LIBS:power
 LIBS:device
@@
 LIBS:contrib
 LIBS:valves
+LIBS:w_connectors
 LIBS: cycloscope_photo_trigger-cache
 EELAYER 25  0
@@
 Sheet 1 1
 Title "Cycloscop photo trigger"
-Date "21 apr 2014"
+Date "25 apr 2014"
 Rev "1"
 Comp "Raspibo"
@@
 $EndDescr
 Wire Wire Line
+	6700 4350 6700 4200
+Wire Wire Line
+	6700 4200 6800 4200
+Connection ~ 6700 4100
+Wire Wire Line
+	6650 4100 6800 4100
+Wire Wire Line
+	7800 4750 7800 4950
+Wire Wire Line
+	7800 4100 7450 4100
+Wire Wire Line
+	7450 4100 7450 3550
+Connection ~ 7800 4100
+Wire Wire Line
+	7450 3550 6000 3550
+Wire Wire Line
+	6000 800  6000 650
+Wire Wire Line
+	6000 650  4500 650
+Wire Wire Line
+	4500 650  4500 850
+Wire Wire Line
+	4500 850  2750 850
+Connection ~ 2750 850
+Wire Wire Line
+	6550 2300 6300 2300
+Connection ~ 2750 2000
+Wire Wire Line
+	2800 4550 2800 4700
+Wire Wire Line
+	6000 3150 6300 3150
+Wire Wire Line
+	6300 3150 6300 3100
+Connection ~ 4000 2100
+Wire Wire Line
+	6000 2500 6550 2500
+Wire Wire Line
+	6250 1750 6000 1750
+Wire Wire Line
+	3700 2650 3700 2550
+Wire Wire Line
+	7650 2850 7650 3050
+Wire Wire Line
+	7650 1750 7650 1850
+Wire Wire Line
+	2750 1400 2750 1500
+Wire Wire Line
+	4000 4750 4000 4300
+Wire Wire Line
+	4000 4300 4100 4300
+Wire Wire Line
+	4100 4400 4000 4400
+Connection ~ 4000 4400
+Wire Wire Line
+	2750 2650 2750 2800
+Wire Wire Line
+	2750 2250 2750 1900
+Connection ~ 2750 2100
+Wire Wire Line
+	7650 2350 7650 2450
+Wire Wire Line
+	3700 2150 3700 2100
+Connection ~ 3700 2100
+Wire Wire Line
+	6000 1350 6000 1300
+Wire Wire Line
+	6000 2100 6000 1950
+Wire Wire Line
+	6000 1950 6250 1950
+Wire Wire Line
+	6000 2400 6550 2400
+Wire Wire Line
+	6000 2600 6550 2600
+Wire Wire Line
+	6000 3250 7650 3250
+Wire Wire Line
+	6800 3900 6000 3900
+Wire Wire Line
+	6300 3500 6300 3550
+Connection ~ 6300 3550
+Connection ~ 3700 2650
+Connection ~ 6000 750
+Connection ~ 4000 4750
+Connection ~ 3700 2650
+Connection ~ 4100 4400
+Connection ~ 4100 4300
+Connection ~ 7650 1750
+Wire Wire Line
+	2750 800  2750 900
+Wire Wire Line
+	4100 2100 2750 2100
+Wire Wire Line
+	4000 2100 4000 2400
+Wire Wire Line
+	4000 2400 4100 2400
+Wire Wire Line
+	6300 2100 6550 2100
+Wire Wire Line
+	3200 1900 3200 2100
+Connection ~ 3200 2100
+Wire Wire Line
+	7800 3450 7800 3550
+Connection ~ 7800 3500
+Connection ~ 7800 4850
+Wire Wire Line
 	7800 4150 7800 4050
-Connection ~ 7800 4850
-Connection ~ 7800 3500
-Wire Wire Line
-	7800 3450 7800 3550
-Connection ~ 3200 2100
-Wire Wire Line
-	3200 1900 3200 2100
-Wire Wire Line
-	6300 2100 6550 2100
-Connection ~ 6600 3750
-Wire Wire Line
-	6500 3750 6600 3750
-Wire Wire Line
-	4100 2400 4000 2400
-Wire Wire Line
-	4000 2400 4000 2100
-Wire Wire Line
-	4100 2100 2750 2100
-Connection ~ 6800 4100
-Connection ~ 6800 3800
-Wire Wire Line
-	2750 800  2750 900
-Connection ~ 6600 3700
-Connection ~ 7650 1750
-Connection ~ 4100 4300
-Connection ~ 4100 4400
-Connection ~ 3700 2650
-Connection ~ 4000 4750
-Connection ~ 6000 750
-Connection ~ 3700 2650
-Connection ~ 6300 3550
-Wire Wire Line
-	6300 3500 6300 3550
-Connection ~ 6600 3800
-Wire Wire Line
-	6600 3700 6600 4100
-Wire Wire Line
-	6600 4100 6800 4100
-Wire Wire Line
-	6800 4200 6700 4200
-Wire Wire Line
-	6700 4200 6700 4350
-Wire Wire Line
-	6800 3900 6000 3900
-Wire Wire Line
-	6000 3250 7650 3250
-Wire Wire Line
-	6000 2600 6550 2600
-Wire Wire Line
-	6000 2400 6550 2400
-Wire Wire Line
-	6250 1950 6000 1950
-Wire Wire Line
-	6000 1950 6000 2100
-Wire Wire Line
-	6000 1350 6000 1300
-Connection ~ 3700 2100
-Wire Wire Line
-	3700 2150 3700 2100
-Wire Wire Line
-	7650 2350 7650 2450
-Connection ~ 2750 2100
-Wire Wire Line
-	2750 2250 2750 1900
-Wire Wire Line
-	2750 2650 2750 2800
-Connection ~ 4000 4400
-Wire Wire Line
-	4100 4400 4000 4400
-Wire Wire Line
-	4100 4300 4000 4300
-Wire Wire Line
-	4000 4300 4000 4750
-Wire Wire Line
-	2750 1400 2750 1500
-Wire Wire Line
-	7650 1750 7650 1850
-Wire Wire Line
-	7650 2850 7650 3050
-Wire Wire Line
-	3700 2650 3700 2550
-Wire Wire Line
-	6250 1750 6000 1750
-Wire Wire Line
-	6000 2500 6550 2500
-Wire Wire Line
-	6800 4000 6000 4000
-Wire Wire Line
-	6800 3800 6600 3800
-Connection ~ 4000 2100
-Wire Wire Line
-	6300 3100 6300 3150
-Wire Wire Line
-	6300 3150 6000 3150
-Wire Wire Line
-	2800 4550 2800 4700
-Wire Wire Line
-	6600 4300 6700 4300
-Connection ~ 6700 4300
-Connection ~ 2750 2000
-Wire Wire Line
-	6550 2300 6300 2300
-Connection ~ 2750 850
-Wire Wire Line
-	2750 850  4500 850
-Wire Wire Line
-	4500 850  4500 650
-Wire Wire Line
-	4500 650  6000 650
-Wire Wire Line
-	6000 650  6000 800
-Wire Wire Line
-	6000 3550 7450 3550
-Connection ~ 7800 4100
-Wire Wire Line
-	7450 3550 7450 4100
-Wire Wire Line
-	7450 4100 7800 4100
-Wire Wire Line
-	7800 4750 7800 4950
+Wire Wire Line
+	6700 4100 6700 4050
+Wire Wire Line
+	2650 2700 2750 2700
+Connection ~ 2750 2700
+$Comp
+L PWR_FLAG #FLG01
+U 1 1 535A8F35
+P 2650 2700
+F 0 "#FLG01" H 2650 2795 30  0001 C CNN
+F 1 "PWR_FLAG" H 2650 2880 30  0000 C CNN
+	1    2650 2700
+	0    -1   -1   0
+$EndComp
+$Comp
+L PWR_FLAG #FLG02
+U 1 1 535A8F10
+P 6650 4100
+F 0 "#FLG02" H 6650 4195 30  0001 C CNN
+F 1 "PWR_FLAG" H 6650 4280 30  0000 C CNN
+	1    6650 4100
+	0    -1   -1   0
+$EndComp
+$Comp
+L VCC #PWR03
+U 1 1 535A8ED5
+P 6700 4050
+F 0 "#PWR03" H 6700 4150 30  0001 C CNN
+F 1 "VCC" H 6700 4150 30  0000 C CNN
+	1    6700 4050
+	1    0    0    -1
+$EndComp
+$Comp
+L GND #PWR04
+U 1 1 535A8ECA
+P 6700 4350
+F 0 "#PWR04" H 6700 4350 30  0001 C CNN
+F 1 "GND" H 6700 4280 30  0001 C CNN
+	1    6700 4350
+	1    0    0    -1
+$EndComp
+NoConn ~ 6000 4000
+$Comp
+L JACK_3.5MM_3PIN J1
+U 1 1 535A8E53
+P 6950 4050
+F 0 "J1" H 6950 4300 60  0000 C CNN
+F 1 "JACK_3.5MM_3PIN" H 6950 3800 60  0000 C CNN
+	1    6950 4050
+	1    0    0    1
+$EndComp
 $Comp
 L SW_PUSH SW1
@@
 $EndComp
 $Comp
-L VCC #PWR01
+L VCC #PWR05
 U 1 1 53554C10
 P 7800 3450
-F 0 "#PWR01" H 7800 3550 30  0001 C CNN
+F 0 "#PWR05" H 7800 3550 30  0001 C CNN
 F 1 "VCC" H 7800 3550 30  0000 C CNN
 	1    7800 3450
@@
 $EndComp
 $Comp
-L VCC #PWR02
+L VCC #PWR06
 U 1 1 534EF267
 P 3200 1900
-F 0 "#PWR02" H 3200 2000 30  0001 C CNN
+F 0 "#PWR06" H 3200 2000 30  0001 C CNN
 F 1 "VCC" H 3200 2000 30  0000 C CNN
 	1    3200 1900
@@
 $EndComp
 $Comp
-L GND #PWR03
+L GND #PWR07
 U 1 1 534ECA96
 P 6300 2300
-F 0 "#PWR03" H 6300 2300 30  0001 C CNN
+F 0 "#PWR07" H 6300 2300 30  0001 C CNN
 F 1 "GND" H 6300 2230 30  0001 C CNN
 	1    6300 2300
@@
 $EndComp
 $Comp
-L VCC #PWR04
+L VCC #PWR08
 U 1 1 534ECA7D
 P 6300 2100
-F 0 "#PWR04" H 6300 2200 30  0001 C CNN
+F 0 "#PWR08" H 6300 2200 30  0001 C CNN
 F 1 "VCC" H 6300 2200 30  0000 C CNN
 	1    6300 2100
 	1    0    0    -1
-$EndComp
-$Comp
-L PWR_FLAG #FLG05
-U 1 1 534EC493
-P 6500 3750
-F 0 "#FLG05" H 6500 3845 30  0001 C CNN
-F 1 "PWR_FLAG" H 6500 3930 30  0000 C CNN
-	1    6500 3750
-	0    -1   -1   0
-$EndComp
-$Comp
-L PWR_FLAG #FLG06
-U 1 1 534EC471
-P 6600 4300
-F 0 "#FLG06" H 6600 4395 30  0001 C CNN
-F 1 "PWR_FLAG" H 6600 4480 30  0000 C CNN
-	1    6600 4300
-	0    -1   -1   0
 $EndComp
 $Comp
@@
 $EndComp
 $Comp
-L GND #PWR07
+L GND #PWR09
 U 1 1 534EB5D5
 P 2800 4700
-F 0 "#PWR07" H 2800 4700 30  0001 C CNN
+F 0 "#PWR09" H 2800 4700 30  0001 C CNN
 F 1 "GND" H 2800 4630 30  0001 C CNN
 	1    2800 4700
@@
 NoConn ~ 6000 2200
 $Comp
-L VCC #PWR08
-U 1 1 534EAF83
-P 6600 3700
-F 0 "#PWR08" H 6600 3800 30  0001 C CNN
-F 1 "VCC" H 6600 3800 30  0000 C CNN
-	1    6600 3700
-	1    0    0    -1
-$EndComp
-$Comp
-L GND #PWR09
-U 1 1 534EAF79
-P 6700 4350
-F 0 "#PWR09" H 6700 4350 30  0001 C CNN
-F 1 "GND" H 6700 4280 30  0001 C CNN
-	1    6700 4350
-	1    0    0    -1
-$EndComp
-$Comp
-L CONN_5 P7
-U 1 1 534EAF54
-P 7200 4000
-F 0 "P7" V 7150 4000 50  0000 C CNN
-F 1 "CONN_5" V 7250 4000 50  0000 C CNN
-F 4 "Ext sensor conn" V 7200 4000 60  0001 C CNN "Descr"
-	1    7200 4000
-	1    0    0    -1
-$EndComp
-$Comp
 L CONN_6 P6
